File: 電子回路設計/腕駆動回路/腕駆動回路.brd (EAGLE design)
At the start: 75 x 75 mm, 34 parts, among them IC1 TC74HC244AF, U1 BTN9990LV, U2 BTN9990LV

Commit message: 腕駆動回路設計完
Parts:
- added C10, C9: 1n, RCL:C0603
- added C8: 100u, 小形アルミニウム電解コンデンサ_MH7シリーズ:CPOL6.3-7_2.5
- added CN3: (no value), jst-xh:B3B-XH-A
- CN2: device jst-xh:B7B-XH-A -> jst-xh:B9B-XH-A
- moved C4 67.7 mm to (-5.00, -3.00), turned to 180 degrees
- moved R3 65.3 mm to (-5.00, -5.00)
- moved R4 63.3 mm to (-9.50, -3.00)
- moved C6 61.6 mm to (-5.00, -7.00)
- moved C5 60.3 mm to (-9.50, -1.00), turned to 180 degrees
- moved C7 59.6 mm to (-9.50, -5.00)
- moved R1 58.3 mm to (-5.00, -1.00)
- moved R2 56.3 mm to (-9.50, 1.00)
- moved C3 55.0 mm to (-17.0, -2.00), flipped to the bottom
- moved C2 54.6 mm to (8.00, -2.50), turned to 180 degrees
- moved R5 50.6 mm to (-22.5, 8.50), flipped to the bottom, turned to 90 degrees
- moved R6 50.6 mm to (-20.5, 8.50), flipped to the bottom, turned to 90 degrees
- moved R7 50.6 mm to (-24.5, 8.50), flipped to the bottom, turned to 90 degrees
- moved C1 48.3 mm to (8.00, 7.50), turned to 180 degrees
- moved RPWM1 39.7 mm to (-24.5, 8.50), turned to 90 degrees
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Connections:
- new net LS1: C9.1, CN2.8, CN3.1
- new net LS2: C10.1, CN2.7, CN3.2
- net GND: now also C10.2, C8.-, C9.2, CN2.9, CN3.3; no longer CN2.7
- net N$1: now also U1.IN; no longer U2.IN
- net N$2: now also U1.INH; no longer U2.INH
- net N$3: now also U2.IN; no longer U1.IN
- net N$4: now also U2.INH; no longer U1.INH
- net VCC: now also C8.+
Routing:
- net VCC: track 0.00 -> 45.7 mm, vias 0 -> 2
- net N$2: track 0.00 -> 38.5 mm
- net IS1_A: track 0.00 -> 37.6 mm, vias 0 -> 1
- net N$1: track 0.00 -> 35.4 mm, vias 0 -> 2
- net LPWM: track 0.00 -> 27.4 mm, vias 0 -> 2
- net EN: track 0.00 -> 25.3 mm, vias 0 -> 2
- net N$4: track 0.00 -> 25.2 mm
- net N$3: track 0.00 -> 24.5 mm
- net IS2_1: track 0.00 -> 22.8 mm, vias 0 -> 3
- net N$10: track 0.00 -> 21.1 mm
- net IS1: track 0.00 -> 19.3 mm
- net RPWM: track 0.00 -> 17.6 mm
- net IS2: track 0.00 -> 14.6 mm
- net N$8: track 0.00 -> 10.2 mm
- net LS2: track 0.00 -> 8.69 mm
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Other:
- board size 75 x 75 mm -> 67 x 58.5 mm

Commit message: add : AMD add res
Parts:
- added R10, R11, R8, R9: 10k, FLE_抵抗器:R1608
- C1, C2, C3: device RCL:C0805 -> 村田製作所_チップセラミックコンデンサ:C3216
- C10, C4, C5, C6, C7, C9: device RCL:C0603 -> 村田製作所_チップセラミックコンデンサ:C1608
- moved C2 0.42 mm to (7.70, -2.80)
- moved C1 0.20 mm to (7.80, 7.50)
Connections:
- new net N$11: R8.2, U1.INH
- new net N$12: R9.2, U1.IN
- new net N$13: R10.2, U2.IN
- new net N$14: R11.2, U2.INH
- net N$1: now also R9.1; no longer U1.IN
- net N$2: now also R8.1; no longer U1.INH
- net N$3: now also R10.1; no longer U2.IN
- net N$4: now also R11.1; no longer U2.INH
Routing:
- net N$11: track 0.00 -> 31.8 mm
- net N$12: track 0.00 -> 31.0 mm, vias 0 -> 2
- net N$2: track 38.5 -> 8.04 mm
- net N$14: track 0.00 -> 29.4 mm, vias 0 -> 2
- net N$13: track 0.00 -> 27.7 mm
- net N$1: track 35.4 -> 8.50 mm, vias 2 -> 0
- net N$4: track 25.2 -> 2.72 mm
- net N$3: track 24.5 -> 2.53 mm
- net IS2_1: track 22.8 -> 25.4 mm
- net VDD: track 0.30 -> 2.72 mm
- net IS1_A: track 37.6 -> 38.2 mm

Commit message: fix : cam data
Other:
- board text added: "C1"
- board text added: "C10"
- board text added: "C2"
- board text added: "C3"
- board text added: "C4"
- board text added: "C5"
- board text added: "C6"
- board text added: "C7"
- board text added: "C8"
- board text added: "C9"
- board text added: "CN1"
- board text added: "CN2"
- board text added: "CN3"
- board text added: "EN1"
- board text added: "IC1"
- board text added: "LPWM1"
- board text added: "R1"
- board text added: "R10"
- board text added: "R11"
- board text added: "R2"
- board text added: "R3"
- board text added: "R4"
- board text added: "R5"
- board text added: "R6"
- board text added: "R7"
- board text added: "R8"
- board text added: "R9"
- board text added: "RPWM1"
Changed lines of the file:
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@@
 <layer number="116" name="Patch_BOT" color="7" fill="1" visible="yes" active="yes"/>
 <layer number="121" name="_tsilk" color="7" fill="1" visible="yes" active="yes"/>
-<layer number="122" name="_bsilk" color="7" fill="1" visible="yes" active="yes"/>
+<layer number="122" name="_bPlace" color="5" fill="1" visible="yes" active="yes"/>
 <layer number="123" name="tTestmark" color="7" fill="1" visible="yes" active="yes"/>
 <layer number="124" name="bTestmark" color="7" fill="1" visible="yes" active="yes"/>
-<layer number="125" name="_tNames" color="7" fill="1" visible="yes" active="yes"/>
-<layer number="126" name="_bNames" color="7" fill="1" visible="yes" active="yes"/>
+<layer number="125" name="_tNames" color="14" fill="1" visible="yes" active="yes"/>
+<layer number="126" name="_bNames" color="5" fill="1" visible="yes" active="yes"/>
 <layer number="127" name="_tValues" color="7" fill="1" visible="yes" active="yes"/>
 <layer number="128" name="_bValues" color="7" fill="1" visible="yes" active="yes"/>
@@
 <hole x="5" y="-18" drill="2.1"/>
 <hole x="17" y="-18" drill="2.1"/>
+<text x="9.070009375" y="6.230009375" size="1.27" layer="125" rot="R180">C1</text>
+<text x="8.970009375" y="-4.06999375" size="1.27" layer="125" rot="R180">C2</text>
+<text x="-12" y="-2.49999375" size="1.27" layer="126" rot="MR0">C3</text>
+<text x="-5.9999875" y="0" size="1.27" layer="125">C4</text>
+<text x="-10.500003125" y="1.999996875" size="1.27" layer="125">C5</text>
+<text x="-3.49999375" y="-7.500009375" size="1.27" layer="125">C6</text>
+<text x="-10.500003125" y="-9.00000625" size="1.27" layer="125">C7</text>
+<text x="-5.9999875" y="-10.00000625" size="1.016" layer="122" rot="MR180">C8</text>
+<text x="-13" y="-18.4999875" size="1.27" layer="126" rot="MR0">C9</text>
+<text x="-12.5" y="-12" size="1.27" layer="126" rot="MR0">C10</text>
+<text x="-8.500009375" y="-20.000009375" size="1.27" layer="125" ratio="10">CN1</text>
+<text x="-18.4999875" y="2.99999375" size="1.27" layer="126" ratio="10" rot="MR90">CN2</text>
+<text x="-18.9999875" y="-8.000009375" size="1.27" layer="125" ratio="10">CN3</text>
+<text x="-20.000009375" y="11.500003125" size="0.8128" layer="125" rot="R90" align="bottom-center">EN1</text>
+<text x="-10.500003125" y="2.49999375" size="1.27" layer="122" rot="MR90">IC1</text>
+<text x="-22.00000625" y="12.5" size="0.8128" layer="125" rot="R90" align="bottom-center">LPWM1</text>
+<text x="-5.9999875" y="1.499996875" size="1.27" layer="125">R1</text>
+<text x="-10.500003125" y="3.49999375" size="1.27" layer="125">R2</text>
+<text x="-3.49999375" y="-5.4999875" size="1.27" layer="125">R3</text>
+<text x="-10.500003125" y="-7.500009375" size="1.27" layer="125">R4</text>
+<text x="-21.86500625" y="7.865009375" size="1.27" layer="126" rot="MR90">R5</text>
+<text x="-19.865009375" y="7.865009375" size="1.27" layer="126" rot="MR90">R6</text>
+<text x="-23.865003125" y="7.865009375" size="1.27" layer="126" rot="MR90">R7</text>
+<text x="-3.39999375" y="-4.150003125" size="0.8128" layer="126" rot="MR180" align="bottom-center">R8</text>
+<text x="-3.39999375" y="-6.35" size="0.8128" layer="126" rot="MR180" align="bottom-center">R9</text>
+<text x="-3.39999375" y="3.69999375" size="0.8128" layer="126" rot="MR180" align="bottom-center">R10</text>
+<text x="-3.39999375" y="5.95" size="0.8128" layer="126" rot="MR180" align="bottom-center">R11</text>
+<text x="-24.000003125" y="12.5" size="0.8128" layer="125" rot="R90" align="bottom-center">RPWM1</text>
 </plain>
 <attributes>
