File: 電子回路設計/足駆動回路/足駆動回路.sch (EAGLE design)
At the start: 44 parts, among them CN1 798-HVH-280-3P-6.5DS, CN3 798-HVH-280-3P-6.5DS, IC1 TC74HC244AF, IC2 TC74HC244AF, U1 BTN9990LV, U2 BTN9990LV, U3 BTN9990LV, U4 BTN9990LV

Commit message: fix : RMD res / add : RMD cam
Parts:
- added R15, R16, R17, R18, R19, R20, R21, R22: 10k, FLE_抵抗器:RC0603J10K
Connections:
- new net N$21: R15.2, U1.INH
- new net N$22: R16.2, U1.IN
- new net N$23: R17.2, U2.INH
- new net N$24: R18.2, U2.IN
- new net N$25: R19.2, U3.IN
- new net N$26: R20.2, U3.INH
- new net N$27: R21.2, U4.IN
- new net N$28: R22.2, U4.INH
- net N$1: now also R18.1; no longer U2.IN
- net N$11: now also R21.1; no longer U4.IN
- net N$12: now also R22.1; no longer U4.INH
- net N$13: now also R19.1; no longer U3.IN
- net N$14: now also R20.1; no longer U3.INH
- net N$2: now also R17.1; no longer U2.INH
- net N$3: now also R16.1; no longer U1.IN
- net N$4: now also R15.1; no longer U1.INH
Changed lines of the file:
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@@
 <setting verticaltext="up"/>
 </settings>
-<grid distance="0.1" unitdist="inch" unit="inch" style="lines" multiple="1" display="yes" altdistance="0.01" altunitdist="inch" altunit="inch"/>
+<grid distance="0.05" unitdist="inch" unit="inch" style="lines" multiple="1" display="yes" altdistance="0.01" altunitdist="inch" altunit="inch"/>
 <layers>
 <layer number="1" name="Top" color="4" fill="1" visible="no" active="no"/>
@@
 <part name="R14" library="RCL" deviceset="R" device="1608" package3d_urn="urn:adsk.eagle:package:23555/3" value="1k"/>
 <part name="SUPPLY36" library="supply2" library_urn="urn:adsk.eagle:library:372" deviceset="GND" device=""/>
+<part name="R15" library="FLE_抵抗器" deviceset="RC0603J" device="" package3d_urn="urn:adsk.eagle:package:38223785/2" technology="10K" value="10k"/>
+<part name="R16" library="FLE_抵抗器" deviceset="RC0603J" device="" package3d_urn="urn:adsk.eagle:package:38223785/2" technology="10K" value="10k"/>
+<part name="R17" library="FLE_抵抗器" deviceset="RC0603J" device="" package3d_urn="urn:adsk.eagle:package:38223785/2" technology="10K" value="10k"/>
+<part name="R18" library="FLE_抵抗器" deviceset="RC0603J" device="" package3d_urn="urn:adsk.eagle:package:38223785/2" technology="10K" value="10k"/>
+<part name="R19" library="FLE_抵抗器" deviceset="RC0603J" device="" package3d_urn="urn:adsk.eagle:package:38223785/2" technology="10K" value="10k"/>
+<part name="R20" library="FLE_抵抗器" deviceset="RC0603J" device="" package3d_urn="urn:adsk.eagle:package:38223785/2" technology="10K" value="10k"/>
+<part name="R21" library="FLE_抵抗器" deviceset="RC0603J" device="" package3d_urn="urn:adsk.eagle:package:38223785/2" technology="10K" value="10k"/>
+<part name="R22" library="FLE_抵抗器" deviceset="RC0603J" device="" package3d_urn="urn:adsk.eagle:package:38223785/2" technology="10K" value="10k"/>
 </parts>
 <sheets>
@@
 <instance part="SUPPLY13" gate="GND" x="130.81" y="232.41" smashed="yes"/>
 <instance part="R3" gate="G$1" x="123.19" y="245.11" smashed="yes">
-<attribute name="NAME" x="119.38" y="246.6086" size="1.778" layer="95"/>
-<attribute name="VALUE" x="119.38" y="241.808" size="1.778" layer="96"/>
+<attribute name="NAME" x="118.11" y="246.38" size="1.778" layer="95"/>
+<attribute name="VALUE" x="124.46" y="246.38" size="1.778" layer="96"/>
 </instance>
 <instance part="C6" gate="G$1" x="115.57" y="241.3" smashed="yes">
@@
 </instance>
 <instance part="R4" gate="G$1" x="123.19" y="218.44" smashed="yes">
-<attribute name="NAME" x="119.38" y="219.9386" size="1.778" layer="95"/>
-<attribute name="VALUE" x="119.38" y="215.138" size="1.778" layer="96"/>
+<attribute name="NAME" x="118.11" y="219.71" size="1.778" layer="95"/>
+<attribute name="VALUE" x="124.46" y="219.71" size="1.778" layer="96"/>
 </instance>
 <instance part="C7" gate="G$1" x="115.57" y="214.63" smashed="yes">
@@
 </instance>
 <instance part="SUPPLY36" gate="GND" x="125.73" y="59.69" smashed="yes"/>
+<instance part="R15" gate="G$1" x="123.19" y="250.19" smashed="yes">
+<attribute name="NAME" x="118.11" y="251.46" size="1.778" layer="95"/>
+<attribute name="VALUE" x="124.46" y="251.46" size="1.778" layer="96"/>
+</instance>
+<instance part="R16" gate="G$1" x="123.19" y="255.27" smashed="yes">
+<attribute name="NAME" x="118.11" y="256.54" size="1.778" layer="95"/>
+<attribute name="VALUE" x="124.46" y="256.54" size="1.778" layer="96"/>
+</instance>
+<instance part="R17" gate="G$1" x="123.19" y="223.52" smashed="yes">
+<attribute name="NAME" x="118.11" y="224.79" size="1.778" layer="95"/>
+<attribute name="VALUE" x="124.46" y="224.79" size="1.778" layer="96"/>
+</instance>
+<instance part="R18" gate="G$1" x="123.19" y="228.6" smashed="yes">
+<attribute name="NAME" x="118.11" y="229.87" size="1.778" layer="95"/>
+<attribute name="VALUE" x="124.46" y="229.87" size="1.778" layer="96"/>
+</instance>
+<instance part="R19" gate="G$1" x="123.19" y="146.05" smashed="yes">
+<attribute name="NAME" x="118.11" y="147.32" size="1.778" layer="95"/>
+<attribute name="VALUE" x="124.46" y="147.32" size="1.778" layer="96"/>
+</instance>
+<instance part="R20" gate="G$1" x="123.19" y="140.97" smashed="yes">
+<attribute name="NAME" x="118.11" y="142.24" size="1.778" layer="95"/>
+<attribute name="VALUE" x="124.46" y="142.24" size="1.778" layer="96"/>
+</instance>
+<instance part="R21" gate="G$1" x="123.19" y="119.38" smashed="yes">
+<attribute name="NAME" x="118.11" y="120.65" size="1.778" layer="95"/>
+<attribute name="VALUE" x="124.46" y="120.65" size="1.778" layer="96"/>
+</instance>
+<instance part="R22" gate="G$1" x="123.19" y="114.3" smashed="yes">
+<attribute name="NAME" x="118.11" y="115.57" size="1.778" layer="95"/>
+<attribute name="VALUE" x="124.46" y="115.57" size="1.778" layer="96"/>
+</instance>
 </instances>
 <busses>
@@
 <segment>
 <pinref part="IC1" gate="G1" pin="Y1"/>
-<pinref part="U2" gate="G$1" pin="IN"/>
-<wire x1="101.6" y1="228.6" x2="137.16" y2="228.6" width="0.1524" layer="91"/>
+<wire x1="101.6" y1="228.6" x2="118.11" y2="228.6" width="0.1524" layer="91"/>
+<pinref part="R18" gate="G$1" pin="1"/>
 </segment>
 </net>
 <net name="N$2" class="0">
 <segment>
-<pinref part="U2" gate="G$1" pin="INH"/>
 <pinref part="IC1" gate="G1" pin="Y2"/>
-<wire x1="137.16" y1="223.52" x2="101.6" y2="223.52" width="0.1524" layer="91"/>
+<wire x1="118.11" y1="223.52" x2="101.6" y2="223.52" width="0.1524" layer="91"/>
+<pinref part="R17" gate="G$1" pin="1"/>
 </segment>
 </net>
@@
 <wire x1="101.6" y1="218.44" x2="102.87" y2="218.44" width="0.1524" layer="91"/>
 <wire x1="102.87" y1="218.44" x2="102.87" y2="255.27" width="0.1524" layer="91"/>
-<pinref part="U1" gate="G$1" pin="IN"/>
-<wire x1="102.87" y1="255.27" x2="137.16" y2="255.27" width="0.1524" layer="91"/>
+<wire x1="102.87" y1="255.27" x2="118.11" y2="255.27" width="0.1524" layer="91"/>
+<pinref part="R16" gate="G$1" pin="1"/>
 </segment>
 </net>
@@
 <wire x1="101.6" y1="213.36" x2="104.14" y2="213.36" width="0.1524" layer="91"/>
 <wire x1="104.14" y1="213.36" x2="104.14" y2="250.19" width="0.1524" layer="91"/>
-<pinref part="U1" gate="G$1" pin="INH"/>
-<wire x1="104.14" y1="250.19" x2="137.16" y2="250.19" width="0.1524" layer="91"/>
+<wire x1="104.14" y1="250.19" x2="118.11" y2="250.19" width="0.1524" layer="91"/>
+<pinref part="R15" gate="G$1" pin="1"/>
 </segment>
 </net>
@@
 <net name="N$11" class="0">
 <segment>
-<pinref part="U4" gate="G$1" pin="IN"/>
-<wire x1="101.6" y1="119.38" x2="137.16" y2="119.38" width="0.1524" layer="91"/>
 <pinref part="IC2" gate="G2" pin="Y1"/>
+<wire x1="101.6" y1="119.38" x2="118.11" y2="119.38" width="0.1524" layer="91"/>
+<pinref part="R21" gate="G$1" pin="1"/>
 </segment>
 </net>
 <net name="N$12" class="0">
 <segment>
-<pinref part="U4" gate="G$1" pin="INH"/>
-<wire x1="137.16" y1="114.3" x2="101.6" y2="114.3" width="0.1524" layer="91"/>
 <pinref part="IC2" gate="G2" pin="Y2"/>
+<wire x1="118.11" y1="114.3" x2="101.6" y2="114.3" width="0.1524" layer="91"/>
+<pinref part="R22" gate="G$1" pin="1"/>
 </segment>
 </net>
@@
 <wire x1="101.6" y1="109.22" x2="105.41" y2="109.22" width="0.1524" layer="91"/>
 <wire x1="105.41" y1="109.22" x2="105.41" y2="146.05" width="0.1524" layer="91"/>
-<pinref part="U3" gate="G$1" pin="IN"/>
-<wire x1="105.41" y1="146.05" x2="137.16" y2="146.05" width="0.1524" layer="91"/>
 <pinref part="IC2" gate="G2" pin="Y3"/>
+<wire x1="105.41" y1="146.05" x2="118.11" y2="146.05" width="0.1524" layer="91"/>
+<pinref part="R19" gate="G$1" pin="1"/>
 </segment>
 </net>
@@
 <wire x1="101.6" y1="104.14" x2="106.68" y2="104.14" width="0.1524" layer="91"/>
 <wire x1="106.68" y1="104.14" x2="106.68" y2="140.97" width="0.1524" layer="91"/>
-<pinref part="U3" gate="G$1" pin="INH"/>
-<wire x1="106.68" y1="140.97" x2="137.16" y2="140.97" width="0.1524" layer="91"/>
 <pinref part="IC2" gate="G2" pin="Y4"/>
+<wire x1="106.68" y1="140.97" x2="118.11" y2="140.97" width="0.1524" layer="91"/>
+<pinref part="R20" gate="G$1" pin="1"/>
 </segment>
 </net>
@@
 </segment>
 </net>
+<net name="N$21" class="0">
+<segment>
+<pinref part="U1" gate="G$1" pin="INH"/>
+<wire x1="128.27" y1="250.19" x2="137.16" y2="250.19" width="0.1524" layer="91"/>
+<pinref part="R15" gate="G$1" pin="2"/>
+</segment>
+</net>
+<net name="N$22" class="0">
+<segment>
+<pinref part="U1" gate="G$1" pin="IN"/>
+<wire x1="128.27" y1="255.27" x2="137.16" y2="255.27" width="0.1524" layer="91"/>
+<pinref part="R16" gate="G$1" pin="2"/>
+</segment>
+</net>
+<net name="N$23" class="0">
+<segment>
+<pinref part="U2" gate="G$1" pin="INH"/>
+<wire x1="137.16" y1="223.52" x2="128.27" y2="223.52" width="0.1524" layer="91"/>
+<pinref part="R17" gate="G$1" pin="2"/>
+</segment>
+</net>
+<net name="N$24" class="0">
+<segment>
+<pinref part="U2" gate="G$1" pin="IN"/>
+<wire x1="128.27" y1="228.6" x2="137.16" y2="228.6" width="0.1524" layer="91"/>
+<pinref part="R18" gate="G$1" pin="2"/>
+</segment>
+</net>
+<net name="N$25" class="0">
+<segment>
+<pinref part="U3" gate="G$1" pin="IN"/>
+<wire x1="128.27" y1="146.05" x2="137.16" y2="146.05" width="0.1524" layer="91"/>
+<pinref part="R19" gate="G$1" pin="2"/>
+</segment>
+</net>
+<net name="N$26" class="0">
+<segment>
+<pinref part="U3" gate="G$1" pin="INH"/>
+<wire x1="128.27" y1="140.97" x2="137.16" y2="140.97" width="0.1524" layer="91"/>
+<pinref part="R20" gate="G$1" pin="2"/>
+</segment>
+</net>
+<net name="N$27" class="0">
+<segment>
+<pinref part="U4" gate="G$1" pin="IN"/>
+<wire x1="128.27" y1="119.38" x2="137.16" y2="119.38" width="0.1524" layer="91"/>
+<pinref part="R21" gate="G$1" pin="2"/>
+</segment>
+</net>
+<net name="N$28" class="0">
+<segment>
+<pinref part="U4" gate="G$1" pin="INH"/>
+<wire x1="137.16" y1="114.3" x2="128.27" y2="114.3" width="0.1524" layer="91"/>
+<pinref part="R22" gate="G$1" pin="2"/>
+</segment>
+</net>
