File: 電子回路設計/レシーバー/レシーバ.brd (EAGLE design)
At the start: 18 x 38 mm, 2 parts

Commit message: fix : cam data
Other:
- board text added: "CN1"
Changed lines of the file:
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@@
 <drawing>
 <settings>
-<setting alwaysvectorfont="yes"/>
+<setting alwaysvectorfont="no"/>
 <setting verticaltext="up"/>
 </settings>
@@
 <layer number="123" name="tTestmark" color="7" fill="1" visible="yes" active="yes"/>
 <layer number="124" name="bTestmark" color="7" fill="1" visible="yes" active="yes"/>
-<layer number="125" name="_tNames" color="7" fill="1" visible="yes" active="yes"/>
+<layer number="125" name="_tNames" color="14" fill="1" visible="yes" active="yes"/>
 <layer number="126" name="_bNames" color="7" fill="1" visible="yes" active="yes"/>
 <layer number="127" name="_tValues" color="7" fill="1" visible="yes" active="yes"/>
@@
 </layers>
 <board>
-<fusionsync huburn="a.cGVyc29uYWw6dWUyY2NlZGVl" projecturn="a.cGVyc29uYWw6dWUyY2NlZGVlIzIwMjExMDIwNDU3NjI1ODc2" f3durn="urn:adsk.wipprod:dm.lineage:5JtfklHCQxGW1Lc7PIcS-Q" pcbguid="ea47ac15-e167-46dc-90c5-8b915aad42ab" lastpulledtime="" lastsyncedchangeguid="" latestrevisionid="65c12ae0-642a-424f-9847-a1b18391e8ed" lastsyncedrevisionid="65c12ae0-642a-424f-9847-a1b18391e8ed" lastboardhashguid="7d821a50-d2d7-a291-26b7-20d0bad773b5" lastpushedtime="2022-06-17T06:34:50Z" linktopcb3d="true"/>
+<fusionsync huburn="a.cGVyc29uYWw6dWUyY2NlZGVl" projecturn="a.cGVyc29uYWw6dWUyY2NlZGVlIzIwMjExMDIwNDU3NjI1ODc2" f3durn="urn:adsk.wipprod:dm.lineage:5JtfklHCQxGW1Lc7PIcS-Q" pcbguid="" lastpulledtime="" lastsyncedchangeguid="" latestrevisionid="65c12ae0-642a-424f-9847-a1b18391e8ed" lastsyncedrevisionid="65c12ae0-642a-424f-9847-a1b18391e8ed" lastboardhashguid="7d821a50-d2d7-a291-26b7-20d0bad773b5" lastpushedtime="2022-06-17T06:34:50Z" linktopcb3d="true"/>
 <plain>
 <wire x1="0" y1="-11.5" x2="0" y2="11.5" width="0" layer="20"/>
@@
 <wire x1="2" y1="-13.5" x2="5" y2="-13.5" width="0" layer="20"/>
 <wire x1="13" y1="-13.5" x2="16" y2="-13.5" width="0" layer="20"/>
+<text x="18.9999875" y="12.4499875" size="1.27" layer="125" ratio="10" rot="R270">CN1</text>
 </plain>
 <attributes>
